Commit message: ros2_ws: recalibrate the mecanum base and tune Nav2 for the basket and camera
Motion and odometry, measured on the floor:
- Motor map and polarity redone after finding that rf2o ran in the lidar's
  frame (its startup TF lookup failed) and the IMU is mounted upside down.
  base.launch.py now feeds rf2o its scans 5 s late so the lookup succeeds;
  the URDF gives the IMU roll pi.
- EKF takes x, y and yaw from rf2o's pose instead of its twist, which was
  reversed (lidar faces backwards) and always zero sideways.
- mecanum_base divides commands by measured speed gains (linear 2.87,
  angular 4.12) so Nav2's speed is the robot's real speed.
- calibrate_motor_mapping.py: new script that solves the motor map from
  measured robot motion; check_motor_mapping.py prints per-wheel inversion.

Nav2:
- Footprint grown for the rear basket, the right-side camera and the blind
  zone in front of the lidar; inflation radius 0.35 to match.
- DWB: min_speed_theta 0.35 to skip the turning deadband, BaseObstacle
  scale 0.3; planner cost_penalty 2.0; recoveries look 0.8 s ahead.
- axis_lock off for navigation and SLAM.
- navigation.launch.py loads maps from the source folder and refuses to
  start without the map; base.launch.py refuses to start a second stack.

Also: teleop key hold 0.6 s for Windows auto-repeat over SSH, and rviz2 with
the Nav2 plugins in the Docker image.

File: ros2_ws/src/simulations/jetacker_description/urdf/mecanum_robot.urdf (robot description, URDF)
Before this commit: robot mecanum_robot, 58 links, 57 joints
Joints:
- joint imu_joint: origin xyz=0 0 0.0265 rpy=0 0 0 -> xyz=0 0 0.0265 rpy=3.14159265358979 0 0
